File: Prototipos/Dimmer #1/ProtDimmer/_autosave-ProtDimmer.kicad_sch (KiCad schematic)
At the start: 22 parts, among them J1 Conn_01x02, J2 Conn_01x02, J3 Conn_01x05, K1 SRD-05VDC-SL-C, Q1 BC548B, Q2 BT137, U1 MOC3021M, U2 EL817

Commit message: Agregar librerias, asignar footprints, comenzar pcb
Connections:
- net 48Vca_L: now also J1.1 (Pin_1); no longer J1.2 (Pin_2)
- net 48Vca_N: now also J1.2 (Pin_2); no longer J1.1 (Pin_1)
Other:
- moved on the sheet: J1
