File: Prototipos/Buck #1/KiCad/buck_converter_final/buck_converter_final.kicad_pcb (KiCad board)
At the start: 2 copper layers, 100 x 100 mm, 25 parts, among them J1 Conn_01x03_Pin, J2 Screw_Terminal_01x02, J3 Screw_Terminal_01x02, Q1 IRF9540NPBF, Q3 NPN

Commit message: Primera versión PCB final Buck
Parts:
- moved R11 37.2 mm to (148.3, 91.7), turned to 180 degrees
- moved R13 26.9 mm to (138.2, 91.7), turned to 180 degrees
- moved J3 21.4 mm to (180.0, 80.9)
- moved R8 19.4 mm to (158.8, 83.7)
- moved R14 18.4 mm to (148.6, 84.0), turned to 180 degrees
- moved C2 17.7 mm to (147.1, 79.8), turned to 180 degrees
- moved J2 17.6 mm to (127.6, 78.5)
- moved C6 17.3 mm to (171.6, 91.7), turned to 90 degrees
- moved C7 17.0 mm to (138.1, 81.8), turned to 180 degrees
- moved Q3 16.6 mm to (135.5, 88.0)
- moved Q1 13.2 mm to (140.5, 76.5), turned to 90 degrees
- moved R9 12.2 mm to (166.3, 87.0), turned to 180 degrees
- moved R7 11.7 mm to (166.5, 80.6), turned to 180 degrees
- moved R12 11.0 mm to (135.3, 71.5)
- moved R10 11.0 mm to (167.8, 90.4), turned to 180 degrees
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Connections:
- J1 pad 2: RETRO_MICRO -> AGND
- J1 pad 3: AGND -> RETRO_MICRO
Routing:
- net PGND: track 0.00 -> 94.1 mm
- net Gate: track 0.00 -> 30.4 mm
- net Net-(J3-Pin_1): track 0.00 -> 21.2 mm
- net RETRO_MICRO: track 0.00 -> 17.0 mm
- net Net-(D1-A): track 0.00 -> 14.5 mm
- net 12V: track 0.00 -> 10.6 mm
- net Net-(R10-Pad1): track 0.00 -> 7.35 mm
- net Net-(Q3-B): track 0.00 -> 6.22 mm
- net Net-(C7-Pad1): track 0.00 -> 4.82 mm
- net PWM_CONTROL: track 0.00 -> 3.89 mm
- net AGND: track 0.00 -> 3.74 mm
- net Net-(R7-Pad2): track 0.00 -> 3.12 mm
- net Net-(C3-Pad1): track 0.00 -> 2.89 mm
- net Net-(C2-Pad1): track 0.00 -> 2.73 mm
- added copper zone on B.Cu, net 12V
- added copper zone on B.Cu, net Gate
- added copper zone on B.Cu, net Net-(D1-A)

Commit message: Mejoras en PCB
Parts:
- R11: value 33k -> 2.2k
- R13: value 1k -> 100k
Routing:
- net Net-(D1-A): track 14.5 -> 34.5 mm
- net 12V: track 10.6 -> 23.4 mm
- added copper zone on B.Cu, net PGND
Other:
- board text added: "NSH"
Changed lines of the file:
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@@
 			)
 		)
-		(property "Value" "33k"
+		(property "Value" "2.2k"
 			(at 3.81 0 0)
 			(layer "F.Fab")
@@
 			)
 		)
-		(property "Value" "1k"
+		(property "Value" "100k"
 			(at 3.81 0 0)
 			(layer "F.Fab")
@@
 		(layer "Edge.Cuts")
 	)
+	(gr_text "NSH"
+		(at 171.7 113.1 0)
+		(layer "B.Cu")
+		(effects
+			(font
+				(face "Back to the future 2002")
+				(size 10 10)
+				(thickness 0.3)
+				(bold yes)
+			)
+			(justify left bottom mirror)
+		)
+		(render_cache "NSH" 0
+			(polygon
+				(pts
+					(xy 168.293422 111.373133) (xy 168.386235 110.199546) (xy 168.514057 108.990701) (xy 168.734891 107.544626)
+					(xy 169.040908 106.065323) (xy 169.455408 104.557536) (xy 170.343841 101.80614) (xy 170.77759 100.622149)
+					(xy 171.149842 99.766713) (xy 171.452743 99.056831) (xy 171.446598 98.972923) (xy 168.566974 98.972923)
+					(xy 162.752163 105.360484) (xy 163.48117 102.997431) (xy 164.033827 101.471528) (xy 164.601167 100.131827)
+					(xy 165.148185 98.972923) (xy 161.623761 98.972923) (xy 160.210205 102.312944) (xy 159.874761 103.243174)
+					(xy 159.498848 104.423813) (xy 159.151988 105.754457) (xy 158.763677 107.674075) (xy 158.456101 109.668457)
+					(xy 158.286793 111.439078) (xy 161.023534 111.439078) (xy 165.40464 106.819225) (xy 165.043161 109.705565)
+					(xy 164.969111 110.389928) (xy 164.939357 111.439078) (xy 168.228087 111.439078)
+				)
+			)
+			(polygon
+				(pts
+					(xy 152.795603 99.012002) (xy 151.65916 99.073558) (xy 150.852944 99.232851) (xy 150.29822 99.459577)
+					(xy 149.810938 99.801316) (xy 149.4369 100.210262) (xy 149.163712 100.693614) (xy 148.841111 101.505994)
+					(xy 148.51769 102.450942) (xy 151.79726 102.450942) (xy 152.064943 101.959462) (xy 152.364346 101.620857)
+					(xy 152.696316 101.404429) (xy 153.070376 101.293841) (xy 153.883604 101.213357) (xy 154.601168 101.219347)
+					(xy 155.041434 101.301231) (xy 155.22378 101.429587) (xy 155.261235 101.596702) (xy 155.181493 101.966335)
+					(xy 154.976081 102.604815) (xy 154.714154 103.221291) (xy 154.501639 103.542707) (xy 154.232019 103.771103)
+					(xy 153.84829 103.961584) (xy 153.327229 104.069049) (xy 152.195987 104.11912) (xy 150.95267 104.167935)
+					(xy 149.631437 104.318789) (xy 148.98579 104.478108) (xy 148.481186 104.728276) (xy 148.090482 105.063691)
+					(xy 147.797173 105.491154) (xy 147.508896 106.155674) (xy 147.248174 107.012051) (xy 147.024755 108.097836)
+					(xy 146.886667 109.210982) (xy 146.880399 109.943655) (xy 146.958199 110.401046) (xy 147.104998 110.670291)
+					(xy 147.409555 110.9441) (xy 147.938481 111.226626) (xy 148.781472 111.511741) (xy 152.693021 111.511741)
+					(xy 153.694837 111.491043) (xy 154.512118 111.359728) (xy 155.176268 111.135842) (xy 155.713854 110.830037)
+					(xy 156.145367 110.444765) (xy 156.483835 109.974069) (xy 156.73369 109.404148) (xy 156.890334 108.714549)
+					(xy 156.96666 107.527529) (xy 153.853175 107.527529) (xy 153.690286 108.340979) (xy 153.575959 108.662037)
+					(xy 153.429356 108.876492) (xy 153.271266 109.025959) (xy 152.853149 109.101132) (xy 150.679239 109.152965)
+					(xy 150.372916 109.043024) (xy 150.167557 108.869364) (xy 150.041604 108.625486) (xy 149.996832 108.285737)
+					(xy 150.058251 107.810851) (xy 150.241743 107.229163) (xy 150.458924 106.848673) (xy 150.701618 106.616101)
+					(xy 150.974162 106.496824) (xy 151.700229 106.37716) (xy 152.880478 106.289829) (xy 155.241085 106.183583)
+					(xy 155.963231 106.093974) (xy 156.52335 105.915839) (xy 156.954448 105.662735) (xy 157.303442 105.305963)
+					(xy 157.637969 104.750753) (xy 157.95157 103.934106) (xy 158.642166 101.771336) (xy 159.095237 100.393196)
+					(xy 159.13738 100.087139) (xy 159.067861 99.811962) (xy 158.879082 99.548726) (xy 158.61418 99.340214)
+					(xy 158.27252 99.181132) (xy 157.836165 99.076116) (xy 157.006769 99.005453) (xy 155.257571 98.972923)
+				)
+			)
+			(polygon
+				(pts
+					(xy 144.089567 111.439078) (xy 144.296655 109.340576) (xy 144.466922 108.103942) (xy 144.685075 107.008534)
+					(xy 144.982885 105.84897) (xy 145.693632 103.490806) (xy 146.080819 102.3334) (xy 146.442236 101.364672)
+					(xy 147.326395 99.051081) (xy 144.960293 99.051081) (xy 143.716486 99.070621) (xy 143.842271 99.09016)
+					(xy 143.12457 100.62196) (xy 142.730966 101.548464) (xy 141.965875 103.713677) (xy 139.102128 103.768021)
+					(xy 139.688728 102.156811) (xy 140.193283 100.946406) (xy 140.711773 99.863661) (xy 141.159874 99.051081)
+					(xy 137.627512 99.051081) (xy 136.763294 100.783901) (xy 136.262805 101.913607) (xy 135.856945 102.98347)
+					(xy 135.439096 104.224755) (xy 135.054928 105.491395) (xy 134.728349 106.692829) (xy 134.455249 107.875736)
+					(xy 134.264288 108.953907) (xy 134.149009 110.070276) (xy 134.10614 111.497697) (xy 137.451046 111.497697)
+					(xy 137.874197 108.478244) (xy 138.064714 107.494882) (xy 138.338258 106.378367) (xy 141.204448 106.378367)
+					(xy 141.018021 107.374605) (xy 140.883879 108.291399) (xy 140.776879 109.364384) (xy 140.626203 111.439078)
+					(xy 144.016905 111.439078)
+				)
+			)
+		)
+	)
 	(segment
 		(start 135.52 88)
@@
 	)
 	(segment
+		(start 151.9 72.61)
+		(end 147.93434 72.61)
+		(width 1.4)
+		(layer "B.Cu")
+		(net 3)
+	)
+	(segment
+		(start 155.95 72.54)
+		(end 151.97 72.54)
+		(width 1.4)
+		(layer "B.Cu")
+		(net 3)
+	)
+	(segment
 		(start 144.6 77.205)
 		(end 144.5 77.105)
@@
 	)
 	(segment
+		(start 147.93434 72.61)
+		(end 144.5 76.04434)
+		(width 1.4)
+		(layer "B.Cu")
+		(net 3)
+	)
+	(segment
+		(start 144.5 76.04434)
+		(end 144.5 77.105)
+		(width 1.4)
+		(layer "B.Cu")
+		(net 3)
+	)
+	(segment
+		(start 142.8 74)
+		(end 142.795 74.005)
+		(width 1)
+		(layer "B.Cu")
+		(net 3)
+	)
+	(segment
+		(start 151.97 72.54)
+		(end 151.9 72.61)
+		(width 1.4)
+		(layer "B.Cu")
+		(net 3)
+	)
+	(segment
+		(start 142.795 74.005)
+		(end 140.5 74.005)
+		(width 1)
+		(layer "B.Cu")
+		(net 3)
+	)
+	(segment
+		(start 144.5 75.7)
+		(end 142.8 74)
+		(width 1)
+		(layer "B.Cu")
+		(net 3)
+	)
+	(segment
+		(start 144.5 77.105)
+		(end 144.5 75.7)
+		(width 1)
+		(layer "B.Cu")
+		(net 3)
+	)
+	(segment
 		(start 147.1 77.16)
 		(end 147.2 77.06)
@@
 	)
 	(segment
+		(start 144.545 69.44)
+		(end 144.5 69.485)
+		(width 1.4)
+		(layer "B.Cu")
+		(net 9)
+	)
+	(segment
+		(start 147.2 69.44)
+		(end 144.545 69.44)
+		(width 1.4)
+		(layer "B.Cu")
+		(net 9)
+	)
+	(segment
 		(start 128.23 78.52)
 		(end 135.3 71.45)
@@
 	)
 	(segment
+		(start 142.52 71.465)
+		(end 144.5 69.485)
+		(width 1.4)
+		(layer "B.Cu")
+		(net 9)
+	)
+	(segment
 		(start 127.6 78.52)
 		(end 128.23 78.52)
@@
 	)
 	(segment
+		(start 140.485 71.45)
+		(end 140.5 71.465)
+		(width 1.4)
+		(layer "B.Cu")
+		(net 9)
+	)
+	(segment
+		(start 135.3 71.45)
+		(end 140.485 71.45)
+		(width 1.4)
+		(layer "B.Cu")
+		(net 9)
+	)
+	(segment
+		(start 140.5 71.465)
+		(end 142.52 71.465)
+		(width 1.4)
+		(layer "B.Cu")
+		(net 9)
+	)
+	(segment
 		(start 145.65 84.05)
 		(end 148.56 84.05)
@@
 		(layer "B.Cu")
 		(hatch edge 0.5)
-		(priority 4)
+		(priority 3)
 		(connect_pads yes
 			(clearance 0.4)
@@
 		(polygon
 			(pts
-				(xy 143.65 86.05) (xy 142.25 81.3) (xy 145.8 84.1)
+				(xy 143.65 86.2) (xy 145.4 84.1) (xy 143.5 82.1)
 			)
 		)
 	)
 	(zone
-		(net 9)
-		(net_name "12V")
+		(net 3)
+		(net_name "Net-(D1-A)")
 		(layer "B.Cu")
 		(hatch edge 0.5)
-		(priority 1)
+		(priority 3)
 		(connect_pads yes
 			(clearance 0.4)
@@
 		(polygon
 			(pts
-				(xy 141.7 72.7) (xy 145.35 70.95) (xy 148.3 70.95) (xy 148.35 68.45) (xy 143.3 68.45) (xy 139.05 70.15)
+				(xy 139.1 72.9) (xy 139.1 75) (xy 141.9 75) (xy 143.3 76.2) (xy 143.3 79.7) (xy 143.7 81) (xy 144.4 81.3)
+				(xy 145.3 81.2) (xy 145.7 80.6) (xy 145.8 80.1) (xy 145.8 76.8) (xy 147.725926 74.8) (xy 155.563159 74.8)
+				(xy 160.3 70.3) (xy 155.6 70.9) (xy 149 70.9) (xy 145.4 72.9)
 			)
 		)
 	)
 	(zone
-		(net 3)
-		(net_name "Net-(D1-A)")
+		(net 9)
+		(net_name "12V")
 		(layer "B.Cu")
 		(hatch edge 0.5)
@@
 		(polygon
 			(pts
-				(xy 146.3 72.8) (xy 149.35 70.95) (xy 156.95 70.95) (xy 156.95 74.343396) (xy 152.4 74.521698) (xy 149.9 74.55)
-				(xy 145.75 76.2) (xy 146.330065 74.694054)
+				(xy 134.966667 72.5) (xy 144.079999 72.5) (xy 148.4 70.7) (xy 148.4 68.2) (xy 138.6 68.2) (xy 136.3 68.8)
+				(xy 135.8 69.1) (xy 133.9 70.9)
 			)
 		)
 	)
 	(zone
-		(net 9)
-		(net_name "12V")
+		(net 1)
+		(net_name "PGND")
 		(layer "B.Cu")
 		(hatch edge 0.5)
 		(connect_pads yes
-			(clearance 0.4)
+			(clearance 0.6)
 		)
 		(min_thickness 0.25)
@@
 		(polygon
 			(pts
-				(xy 141.7 72.7) (xy 134.2 72.7) (xy 134.2 70.15) (xy 141.7 70.15)
-			)
-		)
-	)
-	(zone
-		(net 3)
-		(net_name "Net-(D1-A)")
-		(layer "B.Cu")
-		(hatch edge 0.5)
-		(priority 2)
-		(connect_pads yes
-			(clearance 0.4)
-		)
-		(min_thickness 0.25)
-		(filled_areas_thickness no)
-		(fill yes
-			(thermal_gap 0.5)
-			(thermal_bridge_width 0.5)
-			(island_removal_mode 1)
-			(island_area_min 10)
-		)
-		(polygon
-			(pts
-				(xy 139.3 72.8) (xy 139.3 75.25) (xy 141.85 75.25) (xy 143.85 77.95) (xy 145.15 77.95) (xy 146.330065 74.694054)
-				(xy 146.3 72.8)
-			)
-		)
+				(xy 104.8 32.6) (xy 204.8 32.6) (xy 204.8 132.6) (xy 104.8 132.6)
+			)
+		)

Commit message: Avances PCB convertidor Buck
Parts:
- removed J2: Screw_Terminal_01x02, TerminalBlock_Phoenix:TerminalBlock_Phoenix_MKDS-1,5-2-5.08_1x02_P5.08mm_Horizontal
- added J4: ~, Proyecto_Final:BUS_PCIE_x4_NSH, F.Cu at (108.2, 66.5)
Routing:
- net 12V: track 23.4 -> 12.7 mm
- net PGND: track 94.1 -> 84.9 mm
- removed copper zone on B.Cu, net PGND
Other:
- outline, holes or cut-outs redrawn
- board text removed: "NSH"

Commit message: Avances en PCB final buck, versión 1.1
Parts:
- removed J1: Conn_01x03_Pin, Connector_PinHeader_2.54mm:PinHeader_1x03_P2.54mm_Vertical
- moved C6 55.0 mm to (117.0, 85.0), turned to -90 degrees
- moved R10 40.2 mm to (128.0, 84.8)
- moved R9 38.4 mm to (128.0, 88.2)
- moved C1 37.9 mm to (120.4, 100.0)
- moved R11 33.1 mm to (115.2, 92.4), turned to 0 degrees
- moved J3 29.8 mm to (152.8, 93.0), turned to 90 degrees
- moved R8 27.6 mm to (131.4, 80.8), turned to -90 degrees
- moved R2 26.9 mm to (120.3, 70.7), turned to 0 degrees
- moved L1 25.5 mm to (141.3, 73.4)
- moved D1 24.5 mm to (120.3, 73.5), turned to 0 degrees
- moved C3 23.4 mm to (140.7, 65.0), turned to 90 degrees
- moved R7 22.9 mm to (144.0, 84.8)
- moved R5 21.1 mm to (135.1, 69.7), turned to 0 degrees
- moved C2 18.3 mm to (131.0, 71.0), turned to -90 degrees
- moved D2 18.3 mm to (135.1, 65.6), turned to 180 degrees
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Connections:
- J4 pad 10: RETRO_MICRO -> unconnected-(J4-S4-Pad10)
- J4 pad 26: unconnected-(J4-S20-Pad26) -> PWM_CONTROL
- J4 pad 8: PWM_CONTROL -> RETRO_MICRO
Routing:
- net PGND: track 84.9 -> 0.00 mm
- net 12V: track 12.7 -> 48.0 mm
- net Net-(J3-Pin_1): track 21.2 -> 30.6 mm
- net AGND: track 3.74 -> 10.3 mm
- net Net-(R7-Pad2): track 3.12 -> 8.52 mm
- net Net-(D1-A): track 34.5 -> 29.6 mm
- net PWM_CONTROL: track 3.89 -> 7.32 mm
- net Gate: track 30.4 -> 33.3 mm
- net RETRO_MICRO: track 17.0 -> 14.1 mm
- net Net-(C3-Pad1): track 2.89 -> 5.52 mm
- net Net-(Q3-B): track 6.22 -> 7.73 mm
- net Net-(C7-Pad1): track 4.82 -> 3.67 mm
- added copper zone on B.Cu, net Net-(J3-Pin_1)
- added copper zone on B.Cu, net PGND
- removed copper zone on B.Cu, net Gate
