File: Prototipos/Dimmer #1/KiCAD/ProtDimmer/ProtDimmer.kicad_pcb (KiCad board)
At the start: 2 copper layers, 78.7 x 53.3 mm, 22 parts, among them J1 Conn_01x02, J2 Conn_01x02, J3 Conn_01x05, K1 SRD-05VDC-SL-C, Q1 BC548B, Q2 BT137, U1 MOC3021M, U2 EL817

Commit message: Modificaciones varias para facilitar visualización
Routing:
- net unconnected-(U1-NC-Pad3): vias 2 -> 1
- net UC_RELAY: vias 4 -> 2
- net UC_PHASE: vias 0 -> 17
- net UC_DOUT: vias 2 -> 11
- net Retro_micro: vias 9 -> 1
- net RELAY_T2: vias 2 -> 16
- net PWM_MOSFET: vias 2 -> 1
- net Net-(R7-Pad2): vias 12 -> 10
- net Net-(R10-Pad1): vias 1 -> 0
- net Net-(R1-Pad2): vias 17 -> 11
- net Net-(Q3-B): vias 3 -> 2
- net Net-(Q2-G): vias 2 -> 8
- net Net-(Q1-B): vias 5 -> 12
- net Net-(K1-Pad3): vias 2 -> 20
- net Net-(J3-Pin_1): vias 9 -> 4
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Other:
- board size 78.7 x 53.3 mm -> 76.2 x 53.3 mm
