File: Prototipos/Inversor 555/KiCad/Half Bridge Inverter/Half Bridge Inverter.kicad_sch (KiCad schematic)
At the start: 17 parts, among them Q1 IRF540N, Q2 IRF540N, Q3 BC549, U1 TLC555xD

Commit message: Agregar cambios en esquema
Parts:
- removed C4: C, symbol Device:C
- removed D1, D2: D, symbol Device:D
- added U2: LM7809_TO220, Package_TO_SOT_THT:TO-220-3_Vertical, symbol Regulator_Linear:LM7809_TO220
- C1, C2: footprint (none) -> Capacitor_THT:C_Disc_D3.8mm_W2.6mm_P2.50mm
- C3, C5: value C_Polarized_US -> 1000u; footprint (none) -> Capacitor_THT:C_Radial_D10.0mm_H16.0mm_P5.00mm
- Q1, Q2: value IRF540N -> CSD18534Q5A; symbol Transistor_FET:IRF540N -> Transistor_FET:CSD18534Q5A
- Q3: value BC549 -> BC548; symbol Transistor_BJT:BC549 -> Transistor_BJT:BC548
- R1, R2, R3: footprint (none) -> Resistor_THT:R_Axial_DIN0207_L6.3mm_D2.5mm_P7.62mm_Horizontal
- R4: value R -> 100; footprint (none) -> Resistor_THT:R_Axial_DIN0207_L6.3mm_D2.5mm_P7.62mm_Horizontal
- R5: value R -> 5,6k; footprint (none) -> Resistor_THT:R_Axial_DIN0207_L6.3mm_D2.5mm_P7.62mm_Horizontal
- R6: value R -> 120; footprint (none) -> Resistor_THT:R_Axial_DIN0207_L6.3mm_D2.5mm_P7.62mm_Horizontal
- U1: footprint Package_SO:SOIC-8_3.9x4.9mm_P1.27mm -> Package_DIP:DIP-8_W10.16mm
Connections:
- net Earth: now also Q2.1 (S), Q2.2 (S), U2.2 (GND)
- net at Q3.1 (C), R6.2: now also Q2.4 (G); no longer Q2.1 (G)
- net at Q1.3 (S), R3.1: now also Q1.1 (S), Q1.2 (S), Q2.5 (D); no longer Q2.2 (D)
- net at R4.2: now also Q1.4 (G); no longer Q1.1 (G)
- net VCC renamed VDD
- net VDD: now also U2.1 (VI); no longer C3.1, Q1.2 (D)
- new net: C3.1, Q1.5 (D), U2.3 (VO)
Other:
- moved on the sheet: R3

Commit message: Agregar diseño PCB
Parts:
- added J1: Screw_Terminal_01x02, TerminalBlock_Phoenix:TerminalBlock_Phoenix_MKDS-1,5-2-5.08_1x02_P5.08mm_Horizontal, symbol Connector:Screw_Terminal_01x02
- Q1, Q2: value CSD18534Q5A -> IRF4905; symbol Transistor_FET:CSD18534Q5A -> Transistor_FET:IRF4905
- Q3: footprint Package_TO_SOT_THT:TO-92_Inline -> Package_TO_SOT_THT:TO-92_Inline_Wide
- R2: footprint Resistor_THT:R_Axial_DIN0207_L6.3mm_D2.5mm_P7.62mm_Horizontal -> Potentiometer_THT:Potentiometer_Bourns_3296W_Vertical; symbol Device:R -> Device:R_Trim
Connections:
- net Earth: now also J1.1 (Pin_1); no longer Q2.1 (S), Q2.2 (S)
- net VDD: now also J1.2 (Pin_2)
- net at Q3.1 (C), R6.2: now also Q2.1 (G); no longer Q2.4 (G)
- net at C3.1, U2.3 (VO): now also Q1.2 (D); no longer Q1.5 (D)
- net at R4.2: now also Q1.1 (G); no longer Q1.4 (G)
- new net: Q1.3 (S), Q2.2 (D), R3.1
Changed lines of the file:
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@@
+	)
+	(junction
+		(at 44.45 76.2)
+		(diameter 0)
+		(color 0 0 0 0)
 	)
 	(junction
@@
 	)
 	(junction
+		(at 26.67 53.34)
+		(diameter 0)
+		(color 0 0 0 0)
+	)
+	(junction
 		(at 59.69 76.2)
 		(diameter 0)
@@
 	(wire
 		(pts
+			(xy 20.32 57.15) (xy 26.67 57.15)
+		)
+		(stroke
+			(width 0)
+			(type default)
+		)
+	)
+	(wire
+		(pts
 			(xy 26.67 29.21) (xy 59.69 29.21)
 		)
@@
 	(wire
 		(pts
+			(xy 26.67 57.15) (xy 26.67 53.34)
+		)
+		(stroke
+			(width 0)
+			(type default)
+		)
+	)
+	(wire
+		(pts
 			(xy 147.32 109.22) (xy 153.67 109.22)
 		)
@@
 	(wire
 		(pts
+			(xy 20.32 59.69) (xy 26.67 59.69)
+		)
+		(stroke
+			(width 0)
+			(type default)
+		)
+	)
+	(wire
+		(pts
 			(xy 30.48 43.18) (xy 26.67 43.18)
 		)
@@
 	(wire
 		(pts
+			(xy 26.67 76.2) (xy 44.45 76.2)
+		)
+		(stroke
+			(width 0)
+			(type default)
+		)
+	)
+	(wire
+		(pts
 			(xy 176.53 96.52) (xy 161.29 96.52)
 		)
@@
 		(pts
 			(xy 59.69 27.94) (xy 59.69 29.21)
+		)
+		(stroke
+			(width 0)
+			(type default)
+		)
+	)
+	(wire
+		(pts
+			(xy 26.67 59.69) (xy 26.67 76.2)
 		)
 		(stroke
@@
 			)
 		)
-		(property "Footprint" "Package_TO_SOT_THT:TO-92_Inline"
+		(property "Footprint" "Package_TO_SOT_THT:TO-92_Inline_Wide"
 			(at 163.83 111.125 0)
 			(effects
@@
 	)
 	(symbol
-		(lib_id "Device:R")
+		(lib_id "Device:R_Trim")
 		(at 80.01 38.1 180)
 		(unit 1)
@@
 			)
 		)
-		(property "Footprint" "Resistor_THT:R_Axial_DIN0207_L6.3mm_D2.5mm_P7.62mm_Horizontal"
+		(property "Footprint" "Potentiometer_THT:Potentiometer_Bourns_3296W_Vertical"
 			(at 81.788 38.1 90)
 			(effects
@@
 			)
 		)
-		(property "Description" "Resistor"
+		(property "Description" "Trimmable resistor (preset resistor)"
 			(at 80.01 38.1 0)
 			(effects
@@
 	)
 	(symbol
-		(lib_id "Transistor_FET:CSD18534Q5A")
+		(lib_id "Transistor_FET:IRF4905")
 		(at 181.61 64.77 0)
 		(unit 1)
@@
 			)
 		)
-		(property "Value" "CSD18534Q5A"
+		(property "Value" "IRF4905"
 			(at 187.96 66.0399 0)
 			(effects
@@
 			)
 		)
-		(property "Datasheet" "http://www.ti.com/lit/gpn/csd18534q5a"
+		(property "Datasheet" "http://www.infineon.com/dgdl/irf4905.pdf?fileId=5546d462533600a4015355e32165197c"
 			(at 186.69 68.58 0)
 			(effects
@@
 			)
 		)
-		(property "Description" "50A Id, 60V Vds, NexFET N-Channel Power MOSFET, 9.8mOhm Ron, 17nC Qg(typ), SON8 5x6mm"
+		(property "Description" "-74A Id, -55V Vds, Single P-Channel HEXFET Power MOSFET, 20mOhm Ron, TO-220AB"
 			(at 181.61 64.77 0)
 			(effects
@@
 		)
 		(pin "2"
-		)
-		(pin "4"
-		)
-		(pin "5"
 		)
 		(instances
@@
 				(path "/8fe4964a-9912-49f6-ab4d-d9753d9df11d"
 					(reference "#PWR04")
+					(unit 1)
+				)
+			)
+		)
+	)
+	(symbol
+		(lib_id "Connector:Screw_Terminal_01x02")
+		(at 15.24 59.69 180)
+		(unit 1)
+		(exclude_from_sim no)
+		(in_bom yes)
+		(on_board yes)
+		(dnp no)
+		(fields_autoplaced yes)
+		(property "Reference" "J1"
+			(at 15.24 50.8 0)
+			(effects
+				(font
+					(size 1.27 1.27)
+				)
+			)
+		)
+		(property "Value" "Screw_Terminal_01x02"
+			(at 15.24 53.34 0)
+			(effects
+				(font
+					(size 1.27 1.27)
+				)
+			)
+		)
+		(property "Footprint" "TerminalBlock_Phoenix:TerminalBlock_Phoenix_MKDS-1,5-2-5.08_1x02_P5.08mm_Horizontal"
+			(at 15.24 59.69 0)
+			(effects
+				(font
+					(size 1.27 1.27)
+				)
+				(hide yes)
+			)
+		)
+		(property "Datasheet" "~"
+			(at 15.24 59.69 0)
+			(effects
+				(font
+					(size 1.27 1.27)
+				)
+				(hide yes)
+			)
+		)
+		(property "Description" "Generic screw terminal, single row, 01x02, script generated (kicad-library-utils/schlib/autogen/connector/)"
+			(at 15.24 59.69 0)
+			(effects
+				(font
+					(size 1.27 1.27)
+				)
+				(hide yes)
+			)
+		)
+		(pin "1"
+		)
+		(pin "2"
+		)
+		(instances
+			(project ""
+				(path "/8fe4964a-9912-49f6-ab4d-d9753d9df11d"
+					(reference "J1")
 					(unit 1)
 				)
@@
 	)
 	(symbol
-		(lib_id "Transistor_FET:CSD18534Q5A")
+		(lib_id "Transistor_FET:IRF4905")
 		(at 181.61 96.52 0)
 		(unit 1)
@@
 			)
 		)
-		(property "Value" "CSD18534Q5A"
+		(property "Value" "IRF4905"
 			(at 187.96 97.7899 0)
 			(effects
@@
 			)
 		)
-		(property "Datasheet" "http://www.ti.com/lit/gpn/csd18534q5a"
+		(property "Datasheet" "http://www.infineon.com/dgdl/irf4905.pdf?fileId=5546d462533600a4015355e32165197c"
 			(at 186.69 100.33 0)
 			(effects
@@
 			)
 		)
-		(property "Description" "50A Id, 60V Vds, NexFET N-Channel Power MOSFET, 9.8mOhm Ron, 17nC Qg(typ), SON8 5x6mm"
+		(property "Description" "-74A Id, -55V Vds, Single P-Channel HEXFET Power MOSFET, 20mOhm Ron, TO-220AB"
 			(at 181.61 96.52 0)
 			(effects
@@
 		(pin "3"
 		)
-		(pin "5"
-		)
-		(pin "4"
-		)
 		(instances

Commit message: Modificaciones varias para facilitar visualización
Parts:
- U1: footprint Package_DIP:DIP-8_W10.16mm -> Package_DIP:DIP-8_W7.62mm
Changed lines of the file:
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@@
 			)
 		)
-		(property "Footprint" "Package_DIP:DIP-8_W10.16mm"
+		(property "Footprint" "Package_DIP:DIP-8_W7.62mm"
 			(at 81.28 58.42 0)
 			(effects
